File: filament_transformer_breakout.sch (EAGLE design)
At the start: 0 parts

Commit message: * switched to filament transformer breakout * did some small modifications
Parts:
- added R1, R2, R4, R5: parallel, SquantorRCL:WIRE
- added R3, R6: series, SquantorRCL:WIRE
- added U$1: VPP12-200, SquantorTransformer:VPP12-200
- added U$2, U$3, U$4, U$5, U$6, U$7, U$8, U$9: FASTON_2PIN, SquantorConnectors:FASTON_2PIN
Connections:
- new net N$1: R1.2, R3.2, U$1.PRI1,2, U$3.P$1, U$3.P$2
- new net N$2: R1.1, U$1.PRI2,2, U$5.P$1, U$5.P$2
- new net N$3: R4.2, R6.2, U$1.SEC1,2, U$7.P$1, U$7.P$2
- new net N$4: R2.2, U$1.PRI1,1, U$2.P$1, U$2.P$2
- new net N$5: R2.1, R3.1, U$1.PRI2,1, U$4.P$1, U$4.P$2
- new net N$6: R4.1, U$1.SEC2,2, U$9.P$1, U$9.P$2
- new net N$7: R5.2, U$1.SEC1,1, U$6.P$1, U$6.P$2
- new net N$8: R5.1, R6.1, U$1.SEC2,1, U$8.P$1, U$8.P$2
