File: lpc1114FN28_DIP_breakout/lpc1114FN28_DIP_breakout.sch (EAGLE design)
At the start: 0 parts

Commit message: * made a start on the LPC1114FN28 breakout
Parts:
- added C1, C4: 1u, bart_rcl:C-EUC0805K
- added C2, C3: 22p, SquantorRCL:C-EUC0603K
- added C5, C6: 100n, SquantorRCL:C-EUC0603K
- added JP3: JTAG, SquantorConnectors:PINHD-2X5SMD_1.27_SMD
- added LOGO2: OSHW_LOGO_FILLX0150-NT, ohw-logo:OSHW_LOGO_FILLX0150-NT
- added Q1: 12MHz, bart_crystals:CRYSTALSMD_5.0X3.2
- added R1, R2: 10k, bart_rcl:R-EU_R0603
- added R3: 0, SquantorRCL:R-EU_R0603
- added U$1: LPC1114FN28TURNPINHOLE, SquantorNxp:LPC1114FN28TURNPINHOLE
- added U$2, U$3: TACT_2PINDTSM3, SquantorButtons:TACT_2PINDTSM3
- added U$4, U$5: TACT_2PIN, SquantorButtons:TACT_2PIN
Connections:
- new net PIO0_1: R2.2, U$1.PIO0_1, U$2.1, U$4.1
- new net PIO0_11: U$1.PIO0_11
- new net PIO0_2: U$1.PIO0_2
- new net PIO0_3: U$1.PIO0_3
- new net PIO0_4: U$1.PIO0_4
- new net PIO0_5: U$1.PIO0_5
- new net PIO0_6: U$1.PIO0_6
- new net PIO0_7: U$1.PIO0_7
- new net PIO0_8: U$1.PIO0_8
- new net PIO0_9: U$1.PIO0_9
- new net PIO1_0: U$1.PIO1_0
- new net PIO1_1: U$1.PIO1_1
- new net PIO1_2: U$1.PIO1_2
- new net PIO1_4: U$1.PIO1_4
- new net PIO1_5: U$1.PIO1_5
- new net PIO1_6: U$1.PIO1_6
- new net PIO1_7: U$1.PIO1_7
- new net PIO1_8: U$1.PIO1_8
- new net PIO1_9: U$1.PIO1_9
- new net RESET: JP3.10, R1.2, U$1.RESET/PIO0_0, U$3.1, U$5.1
- new net SWCLK: JP3.4, U$1.SWCLK/PIO0_10
- new net SWDIO: JP3.2, U$1.SWDIO/PIO1_3
- new net VDD: C4.1, C6.1, JP3.1, R1.1, R2.1, U$1.VDD
- new net VDDA: C1.1, C5.1, U$1.VDDA
- new net VSS: C2.2, C3.2, C4.2, C6.2, JP3.3, JP3.5, JP3.9, R3.2, U$1.VSS, U$2.2, U$3.2, U$4.2, U$5.2
- new net VSSA: C1.2, C5.2, R3.1, U$1.VSSA
- new net XTALIN: C2.1, Q1.1, U$1.XTALIN
- new net XTALOUT: C3.1, Q1.2, U$1.XTALOUT
