File: kicad/decoupled_IC_socket_254/decoupled_IC_socket_254.sch (KiCad schematic (older format))
At the start: 24 parts, among them J1 PINS_1X20, J10 Proto, J11 Proto, J12 PINS_1X20, J13 PINS_1X20, J14 Proto, J15 Proto, J16 Proto, J17 Proto, J18 Proto, J19 Proto, J2 Proto, J20 Proto, J21 Proto, J22 Proto, J23 Proto, J24 PINS_1X20, J3 Proto, J4 Proto, J5 Proto, J6 Proto, J7 Proto, J8 Proto, J9 Proto

Commit message: * modified decoupled socket to not use pin 1 headers * changed solder mask clearances
Parts:
- J1, J12, J13, J24: footprint SquantorConnectors:Header-0254-1X20-H015 -> SquantorConnectors:Header-0254-1X20-H015_NO_IDX
Changed lines of the file:
@@
 LIBS:SquantorIC
 LIBS:SquantorProto
+LIBS:decoupled_IC_socket_254-cache
 EELAYER 25 0
 EELAYER END
@@
 F 0 "J1" H 800 3350 60  0000 C CNN
 F 1 "PINS_1X20" H 850 1150 60  0000 C CNN
-F 2 "SquantorConnectors:Header-0254-1X20-H015" H 850 3200 60  0001 C CNN
+F 2 "SquantorConnectors:Header-0254-1X20-H015_NO_IDX" H 850 3200 60  0001 C CNN
 F 3 "" H 850 3200 60  0001 C CNN
 	1    850  2250
@@
 F 0 "J12" H 1900 3350 60  0000 C CNN
 F 1 "PINS_1X20" H 1950 1150 60  0000 C CNN
-F 2 "SquantorConnectors:Header-0254-1X20-H015" H 1950 3200 60  0001 C CNN
+F 2 "SquantorConnectors:Header-0254-1X20-H015_NO_IDX" H 1950 3200 60  0001 C CNN
 F 3 "" H 1950 3200 60  0001 C CNN
 	1    1950 2250
@@
 F 0 "J13" H 2800 3350 60  0000 C CNN
 F 1 "PINS_1X20" H 2850 1150 60  0000 C CNN
-F 2 "SquantorConnectors:Header-0254-1X20-H015" H 2850 3200 60  0001 C CNN
+F 2 "SquantorConnectors:Header-0254-1X20-H015_NO_IDX" H 2850 3200 60  0001 C CNN
 F 3 "" H 2850 3200 60  0001 C CNN
 	1    2850 2250
@@
 F 0 "J24" H 3850 3350 60  0000 C CNN
 F 1 "PINS_1X20" H 3900 1150 60  0000 C CNN
-F 2 "SquantorConnectors:Header-0254-1X20-H015" H 3900 3200 60  0001 C CNN
+F 2 "SquantorConnectors:Header-0254-1X20-H015_NO_IDX" H 3900 3200 60  0001 C CNN
 F 3 "" H 3900 3200 60  0001 C CNN
 	1    3900 2250
