File: kicad/proto_PP_40-bottom/proto_PP_40-bottom.kicad_pcb (KiCad board)
At the start: 2 copper layers, 45.5 x 32 mm, 11 parts, among them J1 PINS_1X12, J2 PINS_1X12, J3 Proto, J4 Proto, J5 Proto, J6 Proto

Commit message: * almost finished PP40 bottom protoboard
Parts:
- removed N1: OHWLOGO, Symbols:OSHW-Symbol_6.7x6mm_SilkScreen
- added C1: C, SquantorRcl:C_0805, F.Cu at (131.4, 114.0)
- added C2: C, SquantorRcl:C_0805, F.Cu at (131.4, 87.9)
- added C4: C, SquantorRcl:C_0805, F.Cu at (165.7, 114.9)
- added C5: C, SquantorRcl:C_0805, F.Cu at (165.7, 87.0)
- added J10: Proto_4pins, SquantorProto:proto-TH-0254-04X01-P010SQ-H008, F.Cu at (148.0, 112.4)
- added J11: Proto_4pins, SquantorProto:proto-TH-0254-04X01-P010SQ-H008, F.Cu at (158.1, 112.4)
- added J12: Proto_4pins, SquantorProto:proto-TH-0254-04X01-P010SQ-H008, F.Cu at (137.8, 112.4)
- added J13: Proto, SquantorProto:proto-SMD-0127-04X04-P010, F.Cu at (130.2, 108.6)
- added J14: Proto, SquantorProto:proto-SMD-0127-04X04-P010, F.Cu at (165.7, 108.6)
- added J16: Proto, SquantorProto:proto-TH-0254-04X04-P010SQ-H008, F.Cu at (158.1, 106.0)
- added J17: Proto, SquantorProto:proto-SMD-0127-04X04-P010, F.Cu at (165.7, 103.5)
- added J19: Proto, SquantorProto:proto-TH-0254-04X04-P010SQ-H008, F.Cu at (158.1, 95.9)
- added J20: Proto, SquantorProto:proto-SMD-0127-04X04-P010, F.Cu at (130.2, 93.3)
- added J21: Proto, SquantorProto:proto-SMD-0127-04X04-P010, F.Cu at (165.7, 98.4)
- added J22: Proto, SquantorProto:proto-SMD-0127-04X04-P010, F.Cu at (165.7, 93.3)
- added J23: USB-ID, SquantorUsb:SquantorUsb-USB-UB-SMD4H, F.Cu at (126.0, 101.0)
- added J7: Proto_4pins, SquantorProto:proto-TH-0254-04X01-P010SQ-H008, F.Cu at (158.1, 89.5)
- added J8: Proto_4pins, SquantorProto:proto-TH-0254-04X01-P010SQ-H008, F.Cu at (137.8, 89.5)
- added J9: Proto_4pins, SquantorProto:proto-TH-0254-04X01-P010SQ-H008, F.Cu at (148.0, 89.5)
- added TP1: testpad, SquantorProto:TESTPAD_SQ_1MM, F.Cu at (125.7, 107.3)
- added TP2: testpad, SquantorProto:TESTPAD_SQ_1MM, F.Cu at (130.2, 98.4)
- added TP3: testpad, SquantorProto:TESTPAD_SQ_1MM, F.Cu at (130.2, 103.5)
- added TP4: testpad, SquantorProto:TESTPAD_SQ_1MM, F.Cu at (130.2, 99.7)
- added TP5: testpad, SquantorProto:TESTPAD_SQ_1MM, F.Cu at (130.2, 101.0)
- added TP6: testpad, SquantorProto:TESTPAD_SQ_1MM, F.Cu at (130.2, 102.2)
- added U1: POWER_JOINER, SquantorRcl:R_0402_hand, F.Cu at (148.0, 103.3)
- added U2: POWER_JOINER, SquantorRcl:R_0402_hand, B.Cu at (148.0, 98.9)
- J5, J6: footprint SquantorProto:proto-TH-0254-04X04-P010SQ-H008 -> SquantorProto:proto-TH-0254-04X04-GAP02-P010SQ-H008
- moved J5 43.5 mm to (148.0, 106.0), turned to 180 degrees
- moved J6 31.8 mm to (148.0, 95.9)
Connections:
- J1 pad 1: (no net) -> Net-(J1-Pad1)
- J1 pad 10: (no net) -> Net-(J1-Pad10)
- J1 pad 11: (no net) -> Net-(J1-Pad11)
- J1 pad 12: (no net) -> Net-(J1-Pad12)
- J1 pad 2: (no net) -> Net-(J1-Pad2)
- J1 pad 3: (no net) -> Net-(J1-Pad3)
- J1 pad 4: (no net) -> Net-(J1-Pad4)
- J1 pad 5: (no net) -> Net-(J1-Pad5)
- J1 pad 6: (no net) -> Net-(J1-Pad6)
- J1 pad 7: (no net) -> Net-(J1-Pad7)
- J1 pad 8: (no net) -> Net-(J1-Pad8)
- J1 pad 9: (no net) -> Net-(J1-Pad9)
- J2 pad 1: (no net) -> Net-(J11-Pad1)
- J2 pad 10: (no net) -> Net-(J12-Pad2)
- J2 pad 11: (no net) -> Net-(J12-Pad3)
- J2 pad 12: (no net) -> Net-(J12-Pad4)
- J2 pad 2: (no net) -> Net-(J11-Pad2)
- J2 pad 3: (no net) -> Net-(J11-Pad3)
- J2 pad 4: (no net) -> Net-(J11-Pad4)
- J2 pad 5: (no net) -> Net-(J10-Pad1)
- J2 pad 6: (no net) -> Net-(J10-Pad2)
- J2 pad 7: (no net) -> Net-(J10-Pad3)
- J2 pad 8: (no net) -> Net-(J10-Pad4)
- J2 pad 9: (no net) -> Net-(J12-Pad1)
Routing:
- net GNDA: track 0.00 -> 27.0 mm, vias 0 -> 2
- net GND: track 0.00 -> 25.8 mm, vias 0 -> 2
- net VDDA: track 0.00 -> 25.5 mm
- net VDD: track 0.00 -> 22.6 mm
- net Net-(J23-PadS): track 0.00 -> 18.1 mm
- net Net-(J23-Pad1): track 0.00 -> 3.42 mm
- net Net-(J23-Pad5): track 0.00 -> 3.39 mm
- net Net-(J23-Pad2): track 0.00 -> 3.16 mm
- net Net-(J23-Pad4): track 0.00 -> 3.14 mm
- net Net-(J23-Pad3): track 0.00 -> 2.90 mm
- net Net-(J12-Pad1): track 0.00 -> 2.70 mm
- net Net-(J11-Pad2): track 0.00 -> 2.70 mm
- net Net-(J10-Pad2): track 0.00 -> 2.70 mm
- net Net-(J10-Pad1): track 0.00 -> 2.70 mm
- net Net-(J12-Pad4): track 0.00 -> 2.70 mm
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- added copper zone on B.Cu, net GND
- added copper zone on B.Cu, net GNDA
- added copper zone on F.Cu, net VDD
- added copper zone on F.Cu, net VDDA
Other:
- rule pad_to_mask_clearance: 0.2 -> 0.1

Commit message: * small updates
Parts:
- J13, J14, J17, J20, J21, J22: footprint SquantorProto:proto-SMD-0127-04X04-P010 -> SquantorProto:proto-SMD-0127-04X04-P010-H006
- moved N2 30.6 mm to (130.4, 101.1)
Routing:
- net Net-(J1-Pad4): track 0.00 -> 2.42 mm

Commit message: * minor silk fixes in both PCB's
Parts:
- N2: value V20171120 -> V20171123
Changed lines of the file:
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@@
   )
   (setup
-    (last_trace_width 1)
+    (last_trace_width 0.1524)
     (user_trace_width 0.1524)
     (user_trace_width 0.2)
@@
       (effects (font (size 1 1) (thickness 0.15)))
     )
-    (fp_text value V20171120 (at 0.02 -0.034 270) (layer B.SilkS)
+    (fp_text value V20171123 (at 0.02 -0.034 270) (layer B.SilkS)
       (effects (font (size 1 1) (thickness 0.15)) (justify mirror))
     )
