File: hardware/PPG_breakout/PPG_breakout.sch (KiCad schematic (older format))
At the start: 7 parts

Commit message: completed schematic
Parts:
- D? (x2): footprint (none) -> SquantorDiodes:KPTR-3216
- D?: footprint (none) -> SquantorDiodes:SFH2440_reverse
- J? (x2): footprint (none) -> Connector_PinHeader_2.54mm:PinHeader_1x04_P2.54mm_Vertical
Connections:
- wire segments 8 -> 14
Changed lines of the file:
@@
 F 0 "J?" H 968 1967 50  0000 C CNN
 F 1 "Conn_01x04" H 968 1876 50  0000 C CNN
-F 2 "" H 1050 1650 50  0001 C CNN
+F 2 "Connector_PinHeader_2.54mm:PinHeader_1x04_P2.54mm_Vertical" H 1050 1650 50  0001 C CNN
 F 3 "~" H 1050 1650 50  0001 C CNN
 	1    1050 1650
@@
 F 0 "J?" H 2068 1325 50  0000 C CNN
 F 1 "Conn_01x04" H 2068 1416 50  0000 C CNN
-F 2 "" H 2150 1750 50  0001 C CNN
+F 2 "Connector_PinHeader_2.54mm:PinHeader_1x04_P2.54mm_Vertical" H 2150 1750 50  0001 C CNN
 F 3 "~" H 2150 1750 50  0001 C CNN
 	1    2150 1750
@@
 $Comp
 L Device:LED D?
-U 1 1 5D279473
-P 1600 2200
-F 0 "D?" V 1639 2083 50  0000 R CNN
-F 1 "LED" V 1548 2083 50  0000 R CNN
-F 2 "" H 1600 2200 50  0001 C CNN
-F 3 "~" H 1600 2200 50  0001 C CNN
-	1    1600 2200
-	1    0    0    -1
-$EndComp
-$Comp
-L Device:LED D?
 U 1 1 5D279E87
 P 1600 2950
-F 0 "D?" V 1639 2833 50  0000 R CNN
-F 1 "LED" V 1548 2833 50  0000 R CNN
-F 2 "" H 1600 2950 50  0001 C CNN
+F 0 "D?" H 1593 3166 50  0000 C CNN
+F 1 "LED" H 1593 3075 50  0000 C CNN
+F 2 "SquantorDiodes:KPTR-3216" H 1600 2950 50  0001 C CNN
 F 3 "~" H 1600 2950 50  0001 C CNN
 	1    1600 2950
@@
 U 1 1 5D27B9AE
 P 1650 2600
-F 0 "D?" V 1646 2522 50  0000 R CNN
-F 1 "D_Photo" V 1555 2522 50  0000 R CNN
-F 2 "" H 1600 2600 50  0001 C CNN
+F 0 "D?" H 1600 2895 50  0000 C CNN
+F 1 "D_Photo" H 1600 2804 50  0000 C CNN
+F 2 "SquantorDiodes:SFH2440_reverse" H 1600 2600 50  0001 C CNN
 F 3 "~" H 1600 2600 50  0001 C CNN
 	1    1650 2600
@@
 Wire Wire Line
 	1750 2950 1800 2950
+Wire Wire Line
+	1250 1550 1300 1550
+Wire Wire Line
+	1300 1650 1250 1650
+Wire Wire Line
+	1250 1750 1300 1750
+Wire Wire Line
+	1900 1550 1950 1550
+Wire Wire Line
+	1950 1650 1900 1650
+Wire Wire Line
+	1900 1750 1950 1750
+$Comp
+L Device:LED D?
+U 1 1 5D279473
+P 1600 2200
+F 0 "D?" H 1593 2416 50  0000 C CNN
+F 1 "LED" H 1593 2325 50  0000 C CNN
+F 2 "SquantorDiodes:KPTR-3216" H 1600 2200 50  0001 C CNN
+F 3 "~" H 1600 2200 50  0001 C CNN
+	1    1600 2200
+	1    0    0    -1
+$EndComp
 $EndSCHEMATC

Commit message: library update
Parts:
- removed N1: OHWLOGO, Symbols:OSHW-Symbol_6.7x6mm_SilkScreen, symbol SquantorLabels:OHWLOGO
- gave numbers to parts that had none: 5
Changed lines of the file:
@@
 $EndComp
 $Comp
-L SquantorLabels:OHWLOGO N1
-U 1 1 5A135869
-P 850 7350
-F 0 "N1" H 850 7500 60  0000 C CNN
-F 1 "OHWLOGO" H 850 7200 60  0000 C CNN
-F 2 "Symbols:OSHW-Symbol_6.7x6mm_SilkScreen" H 850 7350 60  0001 C CNN
-F 3 "" H 850 7350 60  0001 C CNN
-	1    850  7350
-	1    0    0    -1
-$EndComp
-$Comp
-L Connector_Generic:Conn_01x04 J?
+L Connector_Generic:Conn_01x04 J1
 U 1 1 5D277621
 P 1050 1650
-F 0 "J?" H 968 1967 50  0000 C CNN
+F 0 "J1" H 968 1967 50  0000 C CNN
 F 1 "Conn_01x04" H 968 1876 50  0000 C CNN
 F 2 "Connector_PinHeader_2.54mm:PinHeader_1x04_P2.54mm_Vertical" H 1050 1650 50  0001 C CNN
@@
 $EndComp
 $Comp
-L Connector_Generic:Conn_01x04 J?
+L Connector_Generic:Conn_01x04 J2
 U 1 1 5D277F89
 P 2150 1750
-F 0 "J?" H 2068 1325 50  0000 C CNN
+F 0 "J2" H 2068 1325 50  0000 C CNN
 F 1 "Conn_01x04" H 2068 1416 50  0000 C CNN
 F 2 "Connector_PinHeader_2.54mm:PinHeader_1x04_P2.54mm_Vertical" H 2150 1750 50  0001 C CNN
@@
 PD_C
 $Comp
-L Device:LED D?
+L Device:LED D2
 U 1 1 5D279E87
 P 1600 2950
-F 0 "D?" H 1593 3166 50  0000 C CNN
+F 0 "D2" H 1593 3166 50  0000 C CNN
 F 1 "LED" H 1593 3075 50  0000 C CNN
 F 2 "SquantorDiodes:KPTR-3216" H 1600 2950 50  0001 C CNN
@@
 $EndComp
 $Comp
-L Device:D_Photo D?
+L Device:D_Photo D3
 U 1 1 5D27B9AE
 P 1650 2600
-F 0 "D?" H 1600 2895 50  0000 C CNN
+F 0 "D3" H 1600 2895 50  0000 C CNN
 F 1 "D_Photo" H 1600 2804 50  0000 C CNN
 F 2 "SquantorDiodes:SFH2440_reverse" H 1600 2600 50  0001 C CNN
@@
 	1900 1750 1950 1750
 $Comp
-L Device:LED D?
+L Device:LED D1
 U 1 1 5D279473
 P 1600 2200
-F 0 "D?" H 1593 2416 50  0000 C CNN
+F 0 "D1" H 1593 2416 50  0000 C CNN
 F 1 "LED" H 1593 2325 50  0000 C CNN
 F 2 "SquantorDiodes:KPTR-3216" H 1600 2200 50  0001 C CNN
