File: electronics/breakout_sot363/breakout_sot363.kicad_pcb (KiCad board)
At the start: 2 copper layers, 2 parts

Commit message: schematic and routing completed
Parts:
- removed N2: OHWLOGO, Symbol:OSHW-Symbol_6.7x6mm_SilkScreen
- added J1: Conn_01x03, SquantorConnectors:Header-0254-1X03-H010, B.Cu at (147.3, 83.8)
- added J2: Conn_01x03, SquantorConnectors:Header-0254-1X03-H010, B.Cu at (154.9, 83.8)
- added U1: Generic_6pin_IC, SquantorIC:SOT363-NXP-hand, F.Cu at (151.1, 83.8)
- N1: value 20200610 -> 20211107; moved to B.Cu
- moved N1 15.6 mm to (151.3, 83.2), turned to 270 degrees
Routing:
- net Net-(J1-Pad3): track 0.00 -> 3.97 mm
- net Net-(J1-Pad1): track 0.00 -> 3.97 mm
- net Net-(J2-Pad1): track 0.00 -> 3.97 mm
- net Net-(J2-Pad3): track 0.00 -> 3.97 mm
- net Net-(J1-Pad2): track 0.00 -> 2.76 mm
- net Net-(J2-Pad2): track 0.00 -> 2.76 mm
Other:
- board outline added: 10.7 x 8.1 mm
