File: electronics/breakout_SOT457_SOT23-6/breakout_SOT457_SOT23-6.kicad_sch (KiCad schematic)
At the start: 6 parts, among them J1 Conn_01x03, J2 Conn_01x03, U1 Generic_6pin_IC

Commit message: ready for production
Parts:
- N1: value 20240525 -> 20240530
Changed lines of the file:
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@@
       (effects (font (size 1.524 1.524)) (justify left))
     )
-    (property "Value" "20240525" (at 20.32 189.23 0)
+    (property "Value" "20240530" (at 20.32 189.23 0)
       (effects (font (size 1.524 1.524)) (justify left))
     )
