File: electronics/neopixel_RGB_6pin/neopixel_RGB_6pin.kicad_pcb (KiCad board)
At the start: 2 copper layers, 9 x 9 mm, 6 parts, among them J1 Conn_01x03, J2 Conn_01x03

Commit message: production run, updated versionnumbers, added tiled versions
Parts:
- N1: value 20240425 -> 20240712; moved to B.Cu
- moved N1 26.8 mm to (114.5, 78.9), turned to 180 degrees
- moved N2 17.4 mm to (123.5, 79.1)
Changed lines of the file:
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@@
   (net 4 "/Out")
   (net 5 "unconnected-(U1-NC-Pad1)")
-  (footprint "SquantorLabels:Label_Generic" (layer "F.Cu")
-    (at 138.1 91.5)
-    (descr "Label for general purpose use")
-    (tags "Label")
-    (property "Sheetfile" "neopixel_RGB_6pin.kicad_sch")
-    (property "Sheetname" "")
-    (attr smd)
-    (fp_text reference "N1" (at 0 1.85) (layer "F.Fab") hide
-        (effects (font (size 1 1) (thickness 0.15)))
-    )
-    (fp_text value "20240425" (at 0.8 -0.1) (layer "F.SilkS")
-        (effects (font (size 0.8 0.8) (thickness 0.15)))
-    )
-    (fp_line (start -0.5 0.6) (end 0.5 0.6)
-      (stroke (width 0.15) (type solid)) (layer "F.SilkS"))
-  )
   (footprint "Symbol:OSHW-Symbol_6.7x6mm_SilkScreen" (layer "F.Cu")
-    (at 138.7 87.6)
+    (at 123.5 79.1)
     (descr "Open Source Hardware Symbol")
     (tags "Logo Symbol OSHW")
@@
       (net 3 "VSS") (pinfunction "Pin_3") (pintype "passive") (thermal_bridge_angle 45))
   )
+  (footprint "SquantorLabels:Label_Generic" (layer "B.Cu")
+    (at 114.5 78.8875 180)
+    (descr "Label for general purpose use")
+    (tags "Label")
+    (property "Sheetfile" "neopixel_RGB_6pin.kicad_sch")
+    (property "Sheetname" "")
+    (attr smd)
+    (fp_text reference "N1" (at 0 -1.85) (layer "B.Fab") hide
+        (effects (font (size 1 1) (thickness 0.15)) (justify mirror))
+    )
+    (fp_text value "20240712" (at 0 0) (layer "B.SilkS")
+        (effects (font (size 0.8 0.8) (thickness 0.15)) (justify mirror))
+    )
+    (fp_line (start -0.5 -0.6) (end 0.5 -0.6)
+      (stroke (width 0.15) (type solid)) (layer "B.SilkS"))
+  )
   (footprint "SquantorOpto:WS2813E" (layer "B.Cu")
     (at 114.5 75.5 180)
@@
         (effects (font (size 0.8 0.8) (thickness 0.15)) (justify mirror))
     )
-    (fp_text value "~" (at 0 -6.3 unlocked) (layer "B.Fab")
+    (fp_text value "~" (at 0 0 unlocked) (layer "B.Fab")
         (effects (font (size 0.8 0.8) (thickness 0.15)) (justify mirror))
     )
