File: electronics/neopixel_RGB_6pin/neopixel_RGB_6pin.kicad_sch (KiCad schematic)
At the start: 6 parts, among them J1 Conn_01x03, J2 Conn_01x03

Commit message: production run, updated versionnumbers, added tiled versions
Parts:
- N1: value 20240425 -> 20240712
Changed lines of the file:
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@@
       (effects (font (size 1.524 1.524)) (justify left))
     )
-    (property "Value" "20240425" (at 20.32 189.23 0)
+    (property "Value" "20240712" (at 20.32 189.23 0)
       (effects (font (size 1.524 1.524)) (justify left))
     )
@@
     )
   )
+  (symbol (lib_id "power:PWR_FLAG") (at 53.34 181.61 90) (unit 1)
+    (in_bom yes) (on_board yes) (dnp no) (fields_autoplaced)
+    (property "Reference" "#FLG01" (at 51.435 181.61 0)
+      (effects (font (size 1.27 1.27)) hide)
+    )
+    (property "Value" "PWR_FLAG" (at 49.53 181.61 90)
+      (effects (font (size 1.27 1.27)) (justify left))
+    )
+    (property "Footprint" "" (at 53.34 181.61 0)
+      (effects (font (size 1.27 1.27)) hide)
+    )
+    (property "Datasheet" "~" (at 53.34 181.61 0)
+      (effects (font (size 1.27 1.27)) hide)
+    )
+    (pin "1")
+    (instances
+      (project "neopixel_RGB_6pin"
+        (path "/af2fd3c1-3255-4052-a717-1e087a687e67"
+          (reference "#FLG01") (unit 1)
+        )
+      )
+    )
+  )
   (symbol (lib_id "power:VDD") (at 71.12 41.91 270) (unit 1)
     (in_bom yes) (on_board yes) (dnp no)
@@
         (path "/af2fd3c1-3255-4052-a717-1e087a687e67"
           (reference "#PWR07") (unit 1)
+        )
+      )
+    )
+  )
+  (symbol (lib_id "power:PWR_FLAG") (at 53.34 184.15 90) (unit 1)
+    (in_bom yes) (on_board yes) (dnp no) (fields_autoplaced)
+    (property "Reference" "#FLG02" (at 51.435 184.15 0)
+      (effects (font (size 1.27 1.27)) hide)
+    )
+    (property "Value" "PWR_FLAG" (at 49.53 184.15 90)
+      (effects (font (size 1.27 1.27)) (justify left))
+    )
+    (property "Footprint" "" (at 53.34 184.15 0)
+      (effects (font (size 1.27 1.27)) hide)
+    )
+    (property "Datasheet" "~" (at 53.34 184.15 0)
+      (effects (font (size 1.27 1.27)) hide)
+    )
+    (pin "1")
+    (instances
+      (project "neopixel_RGB_6pin"
+        (path "/af2fd3c1-3255-4052-a717-1e087a687e67"
+          (reference "#FLG02") (unit 1)
         )
       )
@@
         )
       )
+    )
+  )
+  (symbol (lib_id "power:VSS") (at 53.34 184.15 270) (unit 1)
+    (in_bom yes) (on_board yes) (dnp no) (fields_autoplaced)
+    (property "Reference" "#PWR06" (at 49.53 184.15 0)
+      (effects (font (size 1.27 1.27)) hide)
+    )
+    (property "Value" "VSS" (at 57.15 184.15 90)
+      (effects (font (size 1.27 1.27)) (justify left))
+    )
+    (property "Footprint" "" (at 53.34 184.15 0)
+      (effects (font (size 1.27 1.27)) hide)
+    )
+    (property "Datasheet" "" (at 53.34 184.15 0)
+      (effects (font (size 1.27 1.27)) hide)
+    )
+    (pin "1")
+    (instances
+      (project "neopixel_RGB_6pin"
+        (path "/af2fd3c1-3255-4052-a717-1e087a687e67"
+          (reference "#PWR06") (unit 1)
+        )
+      )
+    )
+  )
+  (symbol (lib_id "power:VDD") (at 53.34 181.61 270) (unit 1)
+    (in_bom yes) (on_board yes) (dnp no) (fields_autoplaced)
+    (property "Reference" "#PWR05" (at 49.53 181.61 0)
+      (effects (font (size 1.27 1.27)) hide)
+    )
+    (property "Value" "VDD" (at 57.15 181.61 90)
+      (effects (font (size 1.27 1.27)) (justify left))
+    )
+    (property "Footprint" "" (at 53.34 181.61 0)
+      (effects (font (size 1.27 1.27)) hide)
+    )
+    (property "Datasheet" "" (at 53.34 181.61 0)
+      (effects (font (size 1.27 1.27)) hide)
+    )
+    (pin "1")
+    (instances
+      (project "neopixel_RGB_6pin"
+        (path "/af2fd3c1-3255-4052-a717-1e087a687e67"
+          (reference "#PWR05") (unit 1)
+        )
+      )
