File: electronics/module_CH221K_USB-C_PD-sink/module_CH221K_USB-C_PD-sink.kicad_pcb (KiCad board)
At the start: 2 copper layers, 23.5 x 18.2 mm, 20 parts, among them J1 USB-C_PD, J2 Conn_01x02, Q1 PMOS, U1 CH221K

Commit message: review and small changes
Parts:
- DZ2: value VGate -> 8V
- moved N1 1.37 mm to (101.0, 55.6)
- moved N2 1.37 mm to (101.8, 52.1)
Routing:
- net /VBUS: track 25.4 -> 26.9 mm
- net GND: vias 4 -> 5
Changed lines of the file:
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@@
 		(tags "SOD-323")
 		(property "Reference" "DZ2"
-			(at -2.85 -0.9 0)
+			(at -2.95 -0.9 0)
 			(unlocked yes)
 			(layer "F.SilkS")
@@
 			)
 		)
-		(property "Value" "VGate"
-			(at -2.75 -0.9 0)
+		(property "Value" "8V"
+			(at -2.85 0.2 0)
 			(unlocked yes)
-			(layer "F.Fab")
+			(layer "F.SilkS")
 			(effects
 				(font
@@
 		(tags "capacitor 0805 0603 mixed")
 		(property "Reference" "C1"
-			(at 0 -2.2 90)
+			(at -0.3 -2.2 90)
 			(layer "F.SilkS")
 			(effects
@@
 		)
 		(property "Value" "1u"
-			(at 0 -3.2 90)
+			(at -0.3 -3.2 90)
 			(layer "F.SilkS")
 			(effects
@@
 		(tags "capacitor 1206&0805 dual footprint")
 		(property "Reference" "C2"
-			(at 1.6 1.5 0)
+			(at -3 0.3 0)
 			(layer "F.SilkS")
 			(effects
@@
 		)
 		(property "Value" "10u"
-			(at -2.1 1.6 0)
+			(at -3 -2.1 0)
 			(layer "F.SilkS")
 			(effects
@@
 		(tags "resistor 0603")
 		(property "Reference" "R1"
-			(at -1.6 2.3 90)
+			(at -1.2 2.3 90)
 			(layer "F.SilkS")
 			(effects
@@
 		)
 		(property "Value" "1K"
-			(at 0.4 2.3 90)
+			(at 0.9 2.3 90)
 			(layer "F.SilkS")
 			(effects
@@
 	(footprint "SquantorLabels:Label_Generic"
 		(layer "B.Cu")
-		(at 102.2 54.9875 180)
+		(at 101 55.65 180)
 		(descr "Label for general purpose use")
 		(tags "Label")
@@
 		)
 		(property "Value" "20250403"
-			(at 0 0 0)
+			(at 0 -0.0125 0)
 			(layer "B.SilkS")
 			(effects
@@
 	(footprint "Symbol:OSHW-Symbol_6.7x6mm_SilkScreen"
 		(layer "B.Cu")
-		(at 103 51.4375 180)
+		(at 101.8 52.1 180)
 		(descr "Open Source Hardware Symbol")
 		(tags "Logo Symbol OSHW")
@@
 		(property "Footprint" "Symbol:OSHW-Symbol_6.7x6mm_SilkScreen"
 			(at 0 0 0)
+			(unlocked yes)
 			(layer "B.Fab")
 			(hide yes)
@@
 		(property "Datasheet" ""
 			(at 0 0 0)
+			(unlocked yes)
 			(layer "B.Fab")
 			(hide yes)
@@
 		(property "Description" ""
 			(at 0 0 0)
+			(unlocked yes)
 			(layer "B.Fab")
 			(hide yes)
@@
 		(sheetname "Root")
 		(sheetfile "module_CH221K_USB-C_PD-sink.kicad_sch")
-		(attr exclude_from_pos_files)
+		(attr exclude_from_pos_files allow_missing_courtyard)
 		(fp_poly
 			(pts
@@
 	)
 	(via
+		(at 99.7 50.3)
+		(size 0.7)
+		(drill 0.3)
+		(layers "F.Cu" "B.Cu")
+		(free yes)
+		(net 1)
+	)
+	(via
 		(at 96.3 48.2)
 		(size 0.7)
@@
 	)
 	(segment
-		(start 96.3 49.4)
+		(start 96.6 52.92)
+		(end 95.62 52.92)
+		(width 0.6)
+		(layer "B.Cu")
+		(net 3)
+	)
+	(segment
+		(start 95.2 50.8)
+		(end 96.4 49.6)
+		(width 0.6)
+		(layer "B.Cu")
+		(net 3)
+	)
+	(segment
+		(start 96.4 49.6)
 		(end 96.4 49.3)
 		(width 0.6)
@@
 	)
 	(segment
-		(start 96.6 52.92)
-		(end 96.3 52.62)
+		(start 95.62 52.92)
+		(end 95.2 52.5)
 		(width 0.6)
 		(layer "B.Cu")
@@
 	)
 	(segment
-		(start 96.3 52.62)
-		(end 96.3 49.4)
+		(start 95.2 52.5)
+		(end 95.2 50.8)
 		(width 0.6)
 		(layer "B.Cu")
@@
 	)
 	(segment
-		(start 98.35 47.55)
-		(end 98.35 46.8)
+		(start 98.35 45.85)
+		(end 99.1 45.1)
 		(width 0.2)
 		(layer "F.Cu")
@@
 	(segment
 		(start 100.6 49.35)
-		(end 100.15 49.35)
+		(end 100.6 48.4)
 		(width 0.2)
 		(layer "F.Cu")
@@
 	)
 	(segment
-		(start 100.15 49.35)
-		(end 98.35 47.55)
+		(start 98.35 47.45)
+		(end 98.35 46.8)
 		(width 0.2)
 		(layer "F.Cu")
@@
 	)
 	(segment
-		(start 98.35 45.85)
-		(end 99.1 45.1)
+		(start 100 47.8)
+		(end 98.7 47.8)
 		(width 0.2)
 		(layer "F.Cu")
@@
 	)
 	(segment
+		(start 98.7 47.8)
+		(end 98.35 47.45)
+		(width 0.2)
+		(layer "F.Cu")
+		(net 6)
+	)
+	(segment
 		(start 98.35 46.8)
 		(end 98.35 45.85)
 		(width 0.2)
 		(layer "F.Cu")
+		(net 6)
+	)
+	(segment
+		(start 100.6 48.4)
+		(end 100 47.8)
+		(width 0.2)
+		(layer "F.Cu")

Commit message: prepared for production
Parts:
- N1: value 20250403 -> 20250513
Changed lines of the file:
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@@
 			)
 		)
-		(property "Value" "20250403"
+		(property "Value" "20250513"
 			(at 0 -0.0125 0)
 			(layer "B.SilkS")

Commit message: fixed issues and simplified
Parts:
- removed C3: 1n, SquantorCapacitor:C_0603
- removed C4: 10u, SquantorCapacitor:C_1206_0805
- removed DZ1, DZ2: 8V, SquantorDiodes:SOD-323-nexperia-hand
- removed Q1: PMOS, SquantorIC:SOT23-3
- removed R10: PD, SquantorResistor:R_0603_hand
- removed R9: PU, SquantorResistor:R_0603_hand
- added R3: 5K1, SquantorResistor:R_0603_hand, F.Cu at (97.3, 45.8)
- added R4: 5K1, SquantorResistor:R_0603_hand, F.Cu at (98.6, 45.8)
- R11: value 4K7 -> 10K
- moved R12 16.8 mm to (103.0, 45.8)
- moved D3 9.78 mm to (103.0, 53.5), turned to -90 degrees
- moved C2 5.33 mm to (98.6, 53.9), turned to 0 degrees
- moved N1 2.25 mm to (101.0, 53.4)
- moved N2 2.25 mm to (101.8, 49.9)
- moved J1 1.70 mm to (95.2, 49.7)
- moved D2 1.35 mm to (100.1, 45.8), turned to 90 degrees
- moved R11 1.12 mm to (101.6, 45.8), turned to 90 degrees
- moved R1 0.91 mm to (101.6, 53.6)
- moved R2 0.75 mm to (99.4, 52.0)
- moved U1 0.75 mm to (99.4, 49.5)
- moved C1 0.70 mm to (102.5, 49.6)
- moved J2 0.16 mm to (109.2, 51.4)
Connections:
- D2 pad 1: Net-(D2-K) -> /PG
- D2 pad 2: /PG -> Net-(D2-A)
- J2 pad 1: /VOUT -> /VBUS
- R11 pad 2: Net-(D2-K) -> Net-(D2-A)
Routing:
- net /VOUT: track 16.3 -> 0.00 mm
- net Net-(DZ1-K): track 12.7 -> 0.00 mm
- net Net-(DZ2-A): track 6.62 -> 0.00 mm
- net /PG: track 6.80 -> 2.16 mm
- net Net-(D3-K): track 2.98 -> 7.37 mm
- net /VBUS: track 26.9 -> 30.4 mm
- net /CC2: track 3.61 -> 7.06 mm
- net GND: track 6.22 -> 3.42 mm, vias 5 -> 2
- net /CC1: track 3.59 -> 5.62 mm
- net Net-(D2-A): track 0.00 -> 1.50 mm
- net Net-(D2-K): track 1.20 -> 0.00 mm
- net /VDD: track 11.7 -> 12.7 mm
Other:
- board size 23.5 x 18.2 mm -> 23.5 x 12.9 mm
