File: electronics/DIM_powergate_SOIC-8/DIM_powergate_SOT23-6.kicad_pcb (KiCad board)
At the start: 2 copper layers, 15.7 x 13.7 mm, 10 parts, among them J1 Conn_01x04, J2 Conn_01x04, Q2 NMOS, Q3 Q_PMOS_DUAL

Commit message: Reviewed and fixed
Parts:
- J1, J2: value Conn_01x04 -> Conn_01x05
- N1: value 20260103 -> 20260110; moved to B.Cu
- N2: moved to B.Cu
- moved N1 47.3 mm to (133.3, 44.3), turned to 180 degrees
- moved N2 47.3 mm to (133.3, 40.6), turned to 180 degrees
