File: electronics/DIM_powergate_SOIC-8/DIM_powergate_SOIC-8.kicad_sch (KiCad schematic)
At the start: 10 parts, among them J1 Conn_01x05, J2 Conn_01x05, Q2 NMOS, Q3 Q_PMOS_DUAL

Commit message: preparation for production V20260118
Parts:
- N1: value 20260110 -> 20260118
Changed lines of the file:
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@@
 			)
 		)
-		(property "Value" "20260110"
+		(property "Value" "20260118"
 			(at 20.32 189.23 0)
 			(effects
